File: DH-PRR-0/power_mgmt.kicad_sch (KiCad schematic)
At the start: 17 parts, among them SW2 SW_SPDT, U3 BQ24075RGT, U4 TLV75533PDRV, U5 BQ25887RGE

Commit message: alternate power topologies
Parts:
- removed BT2: 7v4 2s, symbol Device:Battery
- added BT1: 7v4, symbol Device:Battery
- added BT2, BT3: 3v7 1s, symbol Device:Battery_Cell
- added C10, C11, C12, C18, C19, C21, C7, C9: 10u, symbol Device:C
- added C16, C22, C23: 1u, symbol Device:C
- added C17: 4u7, symbol Device:C
- added C20, C8: 44u, symbol Device:C
- added C24: u47, symbol Device:C
- added C25: 2u2, symbol Device:C_Polarized
- added D1, D2, D5: LED, symbol Device:LED
- added L2, L3: 1u, symbol Device:L
- added R10, R21, R22, R23, R25, R4, R5, R6, R9: R, symbol Device:R
- added R18, R19, R20, R27: 10k, symbol Device:R
- added R24: 300, symbol Device:R
- added R26, R7, R8: 1k, symbol Device:R
- added TH1, TH2: 10k, symbol Device:Thermistor_NTC
- added U3: BQ25886RGE, Package_DFN_QFN:Texas_RGE0024H_VQFN-24-1EP_4x4mm_P0.5mm_EP2.7x2.7mm, symbol Battery_Management:BQ25886RGE
- added U4: MIC5219-5.0YMM, Package_SO:MSOP-8_3x3mm_P0.65mm, symbol Regulator_Linear:MIC5219-5.0YMM
- renumbered C7 to C13, C8 to C14, C9 to C15, D1 to D3, D2 to D4, R4 to R11, R5 to R12, R6 to R13, R7 to R14, R8 to R15, R9 to R16, R10 to R17, U4 to U5, U3 to U6, U5 to U7
Connections:
- net VBUS is gone; now on net +5V: C13.1, U5.4 (EN), U5.6 (IN), U6.13 (IN)
- net GND: now also U7.19 (GND), U7.20 (GND), U7.25 (GND), BT1.2 (-), BT3.2 (-), C11.2, C12.2, C16.2, C17.1, C18.2, C20.2, C21.2, C22.2, C23.2, C24.2, C25.2, C7.2, C8.1, C9.2, R10.2, R22.2, R23.1, R4.2, R5.2, R6.1, TH1.2, TH2.2, U3.19 (GND), U3.20 (GND), U3.25 (GND), U3.4 (GND), U4.5 (GND), U4.6 (GND), U4.7 (GND), U4.8 (GND)
- net VOUT: now also C12.1, U3.15 (SYS), U3.16 (SYS)
- net V_{SW}: now also U4.1 (EN), U4.2 (IN); no longer U5.1 (OUT)
- net at U7.1 (~{PG}): now also R27.2
- net at U7.10 (CBSET): now also R25.2
- net at U7.11 (REGN): now also C17.2
- net at U7.12 (BTST): now also C19.2
- net at U7.13 (BAT), U7.14 (BAT): now also BT2.1 (+), C21.1
- net at U7.15 (SNS), U7.16 (SNS): now also C20.1
- net at U7.17 (SW), U7.18 (SW): now also C19.1, L3.2
- net at U7.2 (STAT): now also D5.1 (K)
- net at U7.21 (PMID), U7.22 (PMID): now also C18.1, L3.1
- net +5V: now reaches U7.23 (VBUS)
- net +5V: now also C16.1, C22.1, C25.1, C7.1, R21.1, R9.1, U3.23 (VBUS), U4.3 (OUT)
- net PSEL: now reaches U7.24 (PSEL)
- net CD: now reaches U7.3 (CD)
- net SDA: now reaches U7.4 (SDA)
- net SDA: now also R19.2
- net SCL: now reaches U7.5 (SCL)
- net SCL: now also R18.2
- net ~{INT}: now reaches U7.6 (~{INT})
- net ~{INT}: now also R20.2
- net at U7.7 (TS): now also R21.2, R22.1, TH2.1
- net at U7.8 (ILIM): now also R23.2
- net at U7.9 (MID): now also R24.2
- new net: R10.1, R9.2, TH1.1, U3.7 (TS)
- new net: BT2.2 (-), BT3.1 (+), R24.1, R25.1
- new net: R4.1, U3.8 (ILIM)
- new net: C8.2, U3.11 (REGN)
- new net: R6.2, U3.10 (ICHGSET)
- new net: C10.2, U3.12 (BTST)
- new net: BT1.1 (+), C11.1, U3.13 (BAT), U3.14 (BAT)
- new net: C10.1, L2.2, U3.17 (SW), U3.18 (SW)
- new net: D1.1 (K), U3.2 (STAT)
- new net: C9.1, L2.1, U3.21 (PMID), U3.22 (PMID)
- new net: R5.1, U3.6 (VSET)
- new net: D2.1 (K), U3.9 (~{PG})
- new net: D1.2 (A), R7.2
- new net: D5.2 (A), R26.2
- new net: C24.1, U4.4 (BP)
- new net: D2.2 (A), R8.2
- new net +3V3: C23.1, R18.1, R19.1, R20.1, R26.1, R27.1, R7.1, R8.1, U5.1 (OUT)
- new net D+: U3.24 (D+)
- new net D-: U3.1 (D-)
- new net OTG: U3.5 (OTG)
- new net ~{CE}: U3.3 (~{CE})
Other:
- note added: "connected with jumpers"
- note added: "resistor div"
- moved on the sheet: C13, C14, C15, D3, D4, R11, R12, R13, R14, R15, R16, R17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

Commit message: updated journal.md
Parts:
- added U8: TVS0500DRV, Package_SON:WSON-6-1EP_2x2mm_P0.65mm_EP1x1.6mm, symbol Power_Protection:TVS0500DRV
Connections:
- net +5V: now also U8.4 (IN), U8.5 (IN), U8.6 (IN)
- net GND: now also U8.1 (GND), U8.2 (GND), U8.3 (GND), U8.7 (GND)

Commit message: mcu bootmode
Parts:
- removed BT2, BT3: 3v7 1s, symbol Device:Battery_Cell
- removed C13, C15, C17: 4u7, symbol Device:C
- removed C14: 10u, Capacitor_SMD:C_0805_2012Metric, symbol Device:C
- removed C16: 1u, symbol Device:C
- removed C18, C19, C21: 10u, symbol Device:C
- removed C20: 44u, symbol Device:C
- removed D3, D4, D5: LED, symbol Device:LED
- removed L3: 1u, symbol Device:L
- removed R11, R15, R18, R19, R20, R27: 10k, symbol Device:R
- removed R12, R13, R14, R21, R22, R23, R25: R, symbol Device:R
- removed R16, R17, R26: 1k, symbol Device:R
- removed R24: 300, symbol Device:R
- removed TH2: 10k, symbol Device:Thermistor_NTC
- removed U6: BQ24075RGT, Package_DFN_QFN:VQFN-16-1EP_3x3mm_P0.5mm_EP1.6x1.6mm, symbol Battery_Management:BQ24075RGT
- removed U7: BQ25887RGE, Package_DFN_QFN:Texas_RGE0024H_VQFN-24-1EP_4x4mm_P0.5mm_EP2.7x2.7mm, symbol Battery_Management:BQ25887RGE
- renumbered C22 to C13, C23 to C14, C24 to C15, C25 to C16, U8 to U4, U4 to U5, U5 to U6
Other:
- moved on the sheet: BT1, C11, C12

Commit message: i dont remember
Parts:
- SW2: value SW_SPDT -> PWR_IO
Connections:
- net OTG is gone; now on net +3V3: U3.5 (OTG)
- net +5V: no longer R9.1
- net GND: now also C8.2; no longer C8.1
- net VREGN: now reaches U3.11 (REGN)
- net VREGN: now also C8.1, R9.1; no longer C8.2
Other:
- moved on the sheet: BT1, C11, C12, C8, R10, R4, R5, R6, R9, TH1

Commit message: changed usb-spi bridge to host bridge, now functional
Parts:
- renumbered C7 to C10, C8 to C11, C9 to C12, C10 to C13, C11 to C14, C12 to C15, C13 to C16, C14 to C17, C15 to C18, C16 to C19, L2 to L1, R5 to R10, R6 to R11, R7 to R12, R8 to R13, R9 to R14, R10 to R15, R4 to R9, SW2 to SW4
